File: iv-tracer.kicad_sch (KiCad schematic)
At the start: 10 parts, among them J1 Screw_Terminal, Q1 BUZ11, U1 TMCS1108-Q1, U2 MCP4921, U3 Pico

Commit message: update
Parts:
- R2: value 20K -> 10K
Connections:
- net GPIO10: no longer names the net of U3.14 (GPIO10)
- net GPIO11: no longer names the net of U3.15 (GPIO11)
- net GPIO12: no longer names the net of U3.16 (GPIO12)
- net GPIO13: no longer names the net of U3.17 (GPIO13)
- net GPIO6: no longer names the net of U3.9 (GPIO6)
- net GPIO7: no longer names the net of U3.10 (GPIO7)
- net GPIO8: no longer names the net of U3.11 (GPIO8)
- net GPIO9: no longer names the net of U3.12 (GPIO9)
Other:
- note added: "PV VOLTAGE MEASUREMENT SCALE 1/11"
- note removed: "PV VOLTAGE MEASUREMENT SCALE 1/21"
- moved on the sheet: C1, C2, J1, R2, R3, U2, U3
